File: CarPiPowerHat/RTC.kicad_sch (KiCad schematic)
At the start: 5 parts, among them U5 PCF85063AT/AAZ, Y1 X32K768S301

Commit message: doing some traces
Parts:
- C24: LCSC (none) -> C1525
- D15: LCSC (none) -> C37704
- U5: LCSC (none) -> C2157792
- Y1: LCSC (none) -> C479189
Connections:
- net nRTC_INT: no longer names the net of U5.3 (~INT~)
Changed lines of the file:
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@@
   (junction (at 52.07 46.355) (diameter 1.016) (color 0 0 0 0))
   (no_connect (at 95.885 59.055))
-  (no_connect (at 112.522 61.595))
+  (no_connect (at 95.885 61.595))
   (wire (pts (xy 32.512 45.085) (xy 40.64 45.085))
     (stroke (width 0) (type solid) (color 0 0 0 0))
@@
     (stroke (width 0) (type solid) (color 0 0 0 0))
   )
-  (wire (pts (xy 52.07 46.355) (xy 85.852 46.355))
+  (wire (pts (xy 52.07 46.355) (xy 85.725 46.355))
     (stroke (width 0) (type solid) (color 0 0 0 0))
   )
@@
     (stroke (width 0) (type solid) (color 0 0 0 0))
   )
-  (wire (pts (xy 62.23 51.435) (xy 75.692 51.435))
+  (wire (pts (xy 62.23 51.435) (xy 75.565 51.435))
     (stroke (width 0) (type solid) (color 0 0 0 0))
   )
@@
     (stroke (width 0) (type solid) (color 0 0 0 0))
   )
-  (wire (pts (xy 75.692 61.595) (xy 62.23 61.595))
-    (stroke (width 0) (type solid) (color 0 0 0 0))
-  )
-  (wire (pts (xy 85.852 66.675) (xy 85.852 74.295))
-    (stroke (width 0) (type solid) (color 0 0 0 0))
-  )
-  (wire (pts (xy 96.012 61.595) (xy 112.522 61.595))
+  (wire (pts (xy 75.565 61.595) (xy 62.23 61.595))
+    (stroke (width 0) (type solid) (color 0 0 0 0))
+  )
+  (wire (pts (xy 85.725 66.675) (xy 85.725 74.295))
     (stroke (width 0) (type solid) (color 0 0 0 0))
   )
@@
     (stroke (width 0) (type solid) (color 0 0 0 0))
   )
-  (wire (pts (xy 103.632 51.435) (xy 96.012 51.435))
-    (stroke (width 0) (type solid) (color 0 0 0 0))
-  )
-  (wire (pts (xy 103.632 53.975) (xy 96.012 53.975))
+  (wire (pts (xy 103.632 51.435) (xy 95.885 51.435))
+    (stroke (width 0) (type solid) (color 0 0 0 0))
+  )
+  (wire (pts (xy 103.632 53.975) (xy 95.885 53.975))
     (stroke (width 0) (type solid) (color 0 0 0 0))
   )
@@
     (effects (font (size 2.0066 2.0066)) (justify left bottom))
   )
-  (label "nRTC_INT" (at 98.552 61.595 0)
-    (effects (font (size 1.27 1.27)) (justify left bottom))
-  )
   (label "SCL" (at 101.092 51.435 180)
     (effects (font (size 1.27 1.27)) (justify right bottom))
@@
     (pin "1")
   )
-  (symbol (lib_id "power:GND") (at 85.852 74.295 0) (unit 1)
-    (in_bom yes) (on_board yes)
-    (property "Reference" "#PWR0138" (id 0) (at 85.852 80.645 0)
-      (effects (font (size 1.27 1.27)) hide)
-    )
-    (property "Value" "GND" (id 1) (at 85.979 78.6892 0))
-    (property "Footprint" "" (id 2) (at 85.852 74.295 0)
-      (effects (font (size 1.27 1.27)) hide)
-    )
-    (property "Datasheet" "" (id 3) (at 85.852 74.295 0)
+  (symbol (lib_id "power:GND") (at 85.725 74.295 0) (unit 1)
+    (in_bom yes) (on_board yes)
+    (property "Reference" "#PWR0138" (id 0) (at 85.725 80.645 0)
+      (effects (font (size 1.27 1.27)) hide)
+    )
+    (property "Value" "GND" (id 1) (at 85.852 78.6892 0))
+    (property "Footprint" "" (id 2) (at 85.725 74.295 0)
+      (effects (font (size 1.27 1.27)) hide)
+    )
+    (property "Datasheet" "" (id 3) (at 85.725 74.295 0)
       (effects (font (size 1.27 1.27)) hide)
     )
@@
       (effects (font (size 1.27 1.27)) hide)
     )
+    (property "LCSC" "C479189" (id 7) (at 62.23 56.007 90)
+      (effects (font (size 1.27 1.27)) hide)
+    )
     (pin "1")
     (pin "2")
@@
     )
     (property "Field8" "110091611" (id 9) (at 52.07 51.4604 0)
+      (effects (font (size 1.27 1.27)) hide)
+    )
+    (property "LCSC" "C1525" (id 10) (at 52.07 51.4604 0)
       (effects (font (size 1.27 1.27)) hide)
     )
@@
       (effects (font (size 1.27 1.27)) hide)
     )
+    (property "LCSC" "C37704" (id 9) (at 40.64 52.705 90)
+      (effects (font (size 1.27 1.27)) hide)
+    )
     (pin "1")
     (pin "2")
     (pin "3")
   )
-  (symbol (lib_id "Timer_RTC:PCF8563T") (at 85.852 56.515 0) (unit 1)
-    (in_bom yes) (on_board yes)
-    (property "Reference" "U5" (id 0) (at 85.852 41.8084 0))
-    (property "Value" "PCF85063AT/AAZ" (id 1) (at 85.852 44.1198 0))
-    (property "Footprint" "Package_SO:SOIC-8_3.9x4.9mm_P1.27mm" (id 2) (at 85.852 56.515 0)
-      (effects (font (size 1.27 1.27)) hide)
-    )
-    (property "Datasheet" "https://www.nxp.com/docs/en/data-sheet/PCF85063A.pdf" (id 3) (at 85.852 56.515 0)
-      (effects (font (size 1.27 1.27)) hide)
-    )
-    (property "Field4" "Farnell" (id 4) (at 85.852 56.515 0)
-      (effects (font (size 1.27 1.27)) hide)
-    )
-    (property "Field5" "2890042" (id 5) (at 85.852 56.515 0)
-      (effects (font (size 1.27 1.27)) hide)
-    )
-    (property "Field7" "NXP" (id 6) (at 85.852 56.515 0)
-      (effects (font (size 1.27 1.27)) hide)
-    )
-    (property "Field6" "PCF85063AT/AAZ" (id 7) (at 85.852 56.515 0)
-      (effects (font (size 1.27 1.27)) hide)
-    )
-    (property "Part Description" "Real Time Clock (RTC) IC Clock/Calendar I²C, 2-Wire Serial 8-SOIC (0.154\", 3.90mm Width)" (id 8) (at 85.852 56.515 0)
-      (effects (font (size 1.27 1.27)) hide)
-    )
+  (symbol (lib_id "Timer_RTC:PCF8563T") (at 85.725 56.515 0) (unit 1)
+    (in_bom yes) (on_board yes)
+    (property "Reference" "U5" (id 0) (at 85.725 41.8084 0))
+    (property "Value" "PCF85063AT/AAZ" (id 1) (at 85.725 44.1198 0))
+    (property "Footprint" "Package_SO:SOIC-8_3.9x4.9mm_P1.27mm" (id 2) (at 85.725 56.515 0)
+      (effects (font (size 1.27 1.27)) hide)
+    )
+    (property "Datasheet" "https://www.nxp.com/docs/en/data-sheet/PCF85063A.pdf" (id 3) (at 85.725 56.515 0)
+      (effects (font (size 1.27 1.27)) hide)
+    )
+    (property "Field4" "Farnell" (id 4) (at 85.725 56.515 0)
+      (effects (font (size 1.27 1.27)) hide)
+    )
+    (property "Field5" "2890042" (id 5) (at 85.725 56.515 0)
+      (effects (font (size 1.27 1.27)) hide)
+    )
+    (property "Field7" "NXP" (id 6) (at 85.725 56.515 0)
+      (effects (font (size 1.27 1.27)) hide)
+    )
+    (property "Field6" "PCF85063AT/AAZ" (id 7) (at 85.725 56.515 0)
+      (effects (font (size 1.27 1.27)) hide)
+    )
+    (property "Part Description" "Real Time Clock (RTC) IC Clock/Calendar I²C, 2-Wire Serial 8-SOIC (0.154\", 3.90mm Width)" (id 8) (at 85.725 56.515 0)
+      (effects (font (size 1.27 1.27)) hide)
+    )
+    (property "LCSC" "C2157792" (id 9) (at 85.725 56.515 0)
+      (effects (font (size 1.27 1.27)) hide)
+    )
