File: CarPiPowerHat/RTC.kicad_sch (KiCad schematic)
At the start: 5 parts, among them U5 PCF85063AT/AAZ, Y1 X32K768S301

Commit message: Added part numbers
* Selected parts from lcsc
* Checked footprints
Parts:
- C24: value 100n -> 100n 16v
Changed lines of the file:
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@@
       (effects (font (size 1.27 1.27)) (justify left))
     )
-    (property "Value" "100n" (id 1) (at 54.991 52.6034 0)
+    (property "Value" "100n 16v" (id 1) (at 54.991 52.6034 0)
       (effects (font (size 1.27 1.27)) (justify left))
     )

Commit message: Fixed some bugs, not done yet
Parts:
- BT1: Mouser No (none) -> 534-3034
- Y1: value X32K768S301 -> FC-12M32.768KHZ7PF20PPM; Field6 X32K768S301 -> FC-12M32.768KHZ7PF20PPM; Field7 AEL -> Seiko Epson; LCSC C479189 -> C99009
- renumbered C24 to C1, D15 to D1, U5 to U1
Other:
- moved on the sheet: Y1
Changed lines of the file:
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@@
     (stroke (width 0) (type solid) (color 0 0 0 0))
   )
-  (wire (pts (xy 62.23 51.435) (xy 62.23 53.467))
-    (stroke (width 0) (type solid) (color 0 0 0 0))
-  )
-  (wire (pts (xy 62.23 51.435) (xy 75.565 51.435))
-    (stroke (width 0) (type solid) (color 0 0 0 0))
-  )
-  (wire (pts (xy 62.23 61.595) (xy 62.23 58.547))
-    (stroke (width 0) (type solid) (color 0 0 0 0))
-  )
-  (wire (pts (xy 75.565 61.595) (xy 62.23 61.595))
+  (wire (pts (xy 67.31 51.435) (xy 67.31 53.467))
+    (stroke (width 0) (type solid) (color 0 0 0 0))
+  )
+  (wire (pts (xy 67.31 51.435) (xy 75.565 51.435))
+    (stroke (width 0) (type solid) (color 0 0 0 0))
+  )
+  (wire (pts (xy 67.31 61.595) (xy 67.31 58.547))
+    (stroke (width 0) (type solid) (color 0 0 0 0))
+  )
+  (wire (pts (xy 75.565 61.595) (xy 67.31 61.595))
     (stroke (width 0) (type solid) (color 0 0 0 0))
   )
@@
     (pin "1")
   )
-  (symbol (lib_id "Device:Crystal_Small") (at 62.23 56.007 90) (unit 1)
-    (in_bom yes) (on_board yes)
-    (property "Reference" "Y1" (id 0) (at 64.4652 54.864 90)
+  (symbol (lib_id "Device:Crystal_Small") (at 67.31 56.007 90) (unit 1)
+    (in_bom yes) (on_board yes)
+    (property "Reference" "Y1" (id 0) (at 69.5452 54.864 90)
       (effects (font (size 1.27 1.27)) (justify right))
     )
-    (property "Value" "X32K768S301" (id 1) (at 64.4652 57.15 90)
+    (property "Value" "FC-12M32.768KHZ7PF20PPM" (id 1) (at 56.2102 67.945 90)
       (effects (font (size 1.27 1.27)) (justify right))
     )
-    (property "Footprint" "Crystal:Crystal_SMD_3215-2Pin_3.2x1.5mm" (id 2) (at 62.23 56.007 0)
-      (effects (font (size 1.27 1.27)) hide)
-    )
-    (property "Datasheet" "~" (id 3) (at 62.23 56.007 0)
-      (effects (font (size 1.27 1.27)) hide)
-    )
-    (property "Field6" "X32K768S301" (id 4) (at 62.23 56.007 0)
-      (effects (font (size 1.27 1.27)) hide)
-    )
-    (property "Field7" "AEL" (id 5) (at 62.23 56.007 0)
-      (effects (font (size 1.27 1.27)) hide)
-    )
-    (property "Part Description" "Crystal 32.768KHz 7pF 20pmm" (id 6) (at 62.23 56.007 0)
-      (effects (font (size 1.27 1.27)) hide)
-    )
-    (property "LCSC" "C479189" (id 7) (at 62.23 56.007 90)
+    (property "Footprint" "Crystal:Crystal_SMD_3215-2Pin_3.2x1.5mm" (id 2) (at 67.31 56.007 0)
+      (effects (font (size 1.27 1.27)) hide)
+    )
+    (property "Datasheet" "~" (id 3) (at 67.31 56.007 0)
+      (effects (font (size 1.27 1.27)) hide)
+    )
+    (property "Field6" "FC-12M32.768KHZ7PF20PPM" (id 4) (at 67.31 56.007 0)
+      (effects (font (size 1.27 1.27)) hide)
+    )
+    (property "Field7" "Seiko Epson" (id 5) (at 67.31 56.007 0)
+      (effects (font (size 1.27 1.27)) hide)
+    )
+    (property "Part Description" "Crystal 32.768KHz 7pF 20pmm" (id 6) (at 67.31 56.007 0)
+      (effects (font (size 1.27 1.27)) hide)
+    )
+    (property "LCSC" "C99009" (id 7) (at 67.31 56.007 90)
       (effects (font (size 1.27 1.27)) hide)
     )
@@
       (effects (font (size 1.27 1.27)) hide)
     )
+    (property "Mouser No" "534-3034" (id 9) (at 40.64 65.405 0)
+      (effects (font (size 1.27 1.27)) hide)
+    )
     (pin "1")
     (pin "2")
@@
   (symbol (lib_id "Device:C") (at 52.07 51.4604 0) (unit 1)
     (in_bom yes) (on_board yes)
-    (property "Reference" "C24" (id 0) (at 54.991 50.292 0)
+    (property "Reference" "C1" (id 0) (at 54.991 50.292 0)
       (effects (font (size 1.27 1.27)) (justify left))
     )
@@
   (symbol (lib_id "Diode:BAT54C") (at 40.64 52.705 90) (unit 1)
     (in_bom yes) (on_board yes)
-    (property "Reference" "D15" (id 0) (at 38.4302 51.562 90)
+    (property "Reference" "D1" (id 0) (at 38.4302 51.562 90)
       (effects (font (size 1.27 1.27)) (justify left))
     )
@@
   (symbol (lib_id "Timer_RTC:PCF8563T") (at 85.725 56.515 0) (unit 1)
     (in_bom yes) (on_board yes)
-    (property "Reference" "U5" (id 0) (at 85.725 41.8084 0))
+    (property "Reference" "U1" (id 0) (at 85.725 41.8084 0))
     (property "Value" "PCF85063AT/AAZ" (id 1) (at 85.725 44.1198 0))
     (property "Footprint" "Package_SO:SOIC-8_3.9x4.9mm_P1.27mm" (id 2) (at 85.725 56.515 0)

Commit message: Moved HDMI ports
The HDMI ports were offset by 1-2 mm
Parts:
- U1: Field4 Farnell -> (none); Field5 2890042 -> (none); Field6 PCF85063AT/AAZ -> PCF8563T/5,518; LCSC C2157792 -> C7440
Changed lines of the file:
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@@
       (effects (font (size 1.27 1.27)) hide)
     )
-    (property "Datasheet" "https://www.nxp.com/docs/en/data-sheet/PCF85063A.pdf" (id 3) (at 85.725 56.515 0)
+    (property "Datasheet" "https://datasheet.lcsc.com/lcsc/1809141212_NXP-Semicon-PCF8563T-5,518_C7440.pdf" (id 3) (at 85.725 56.515 0)
       (effects (font (size 1.27 1.27)) hide)
     )
-    (property "Field4" "Farnell" (id 4) (at 85.725 56.515 0)
+    (property "Field4" "" (id 4) (at 85.725 56.515 0)
       (effects (font (size 1.27 1.27)) hide)
     )
-    (property "Field5" "2890042" (id 5) (at 85.725 56.515 0)
+    (property "Field5" "" (id 5) (at 85.725 56.515 0)
       (effects (font (size 1.27 1.27)) hide)
     )
@@
       (effects (font (size 1.27 1.27)) hide)
     )
-    (property "Field6" "PCF85063AT/AAZ" (id 7) (at 85.725 56.515 0)
+    (property "Field6" "PCF8563T/5,518" (id 7) (at 85.725 56.515 0)
       (effects (font (size 1.27 1.27)) hide)
     )
@@
       (effects (font (size 1.27 1.27)) hide)
     )
-    (property "LCSC" "C2157792" (id 9) (at 85.725 56.515 0)
+    (property "LCSC" "C7440" (id 9) (at 85.725 56.515 0)
       (effects (font (size 1.27 1.27)) hide)
     )
