File: CarPiPowerHat/i2s_dac.kicad_sch (KiCad schematic)
At the start: 24 parts, among them J8 AudioJack2_Ground, Q4 DMG2305, U7 AP2112-3.3K, U8 UDA1334ATS

Commit message: doing some traces
Parts:
- removed SJ1: SOLDERJUMPER_CLOSED, SOLDERJUMPER_CLOSEDWIRE, symbol Adafruit I2S Audio UDA1334 Bonnet-eagle-import:SOLDERJUMPER_CLOSED
- C27, C30, C32: footprint 0603-NO -> Capacitor_SMD:C_0603_1608Metric; symbol Adafruit I2S Audio UDA1334 Bonnet-eagle-import:CAP_CERAMIC0603_NO -> Device:C; LCSC (none) -> C14663
- C28, C31: footprint 0805-NO -> Capacitor_SMD:C_0805_2012Metric_Pad1.18x1.45mm_HandSolder
- C29: footprint 0805-NO -> Capacitor_SMD:C_0805_2012Metric; symbol Adafruit I2S Audio UDA1334 Bonnet-eagle-import:CAP_CERAMIC0805-NOOUTLINE -> Device:C; LCSC (none) -> C15850
- C33: footprint PANASONIC_C -> Capacitor_SMD:CP_Elec_6.3x7.7; symbol Adafruit I2S Audio UDA1334 Bonnet-eagle-import:CAP_ELECTROLYTICPANASONIC_C -> Device:C_Polarized; LCSC (none) -> C164078; Mouser (none) -> 647-UCD1H470MCL1GS
- C34: footprint PANASONIC_C -> Capacitor_SMD:CP_Elec_6.3x7.7; symbol Adafruit I2S Audio UDA1334 Bonnet-eagle-import:CAP_ELECTROLYTICPANASONIC_C -> Device:C_Polarized; LCSC (none) -> C134775; Mouser (none) -> 647-UCD1H470MCL1GS
- C35: footprint 0805-NO -> Capacitor_SMD:C_0805_2012Metric; LCSC (none) -> C15850
- C36, C37: footprint 0603-NO -> Capacitor_SMD:C_0603_1608Metric; symbol Adafruit I2S Audio UDA1334 Bonnet-eagle-import:CAP_CERAMIC0603_NO -> Device:C; LCSC (none) -> C57112
- FB1, FB4: footprint 0805 -> Resistor_SMD:R_0805_2012Metric; LCSC (none) -> C1017
- J8: symbol Connector:AudioJack2_Ground -> Connector:AudioJack3_Ground; Mouser (none) -> 490-SJ3524-SMT-TR-GR
- Q4: footprint SOT23-WIDE -> Package_TO_SOT_SMD:SOT-23W_Handsoldering; LCSC (none) -> C144153; Mouser (none) -> 621-DMG2305UX-7
- R22: footprint 0603-NO -> Resistor_SMD:R_0603_1608Metric; symbol Adafruit I2S Audio UDA1334 Bonnet-eagle-import:RESISTOR_0603_NOOUT -> Device:R; LSCSC (none) -> C25804
- R23: footprint 0603-NO -> Resistor_SMD:R_0603_1608Metric_Pad0.98x0.95mm_HandSolder; symbol Adafruit I2S Audio UDA1334 Bonnet-eagle-import:RESISTOR_0603_NOOUT -> Device:R; LCSC (none) -> C25804
- R24, R25: footprint 0603-NO -> Resistor_SMD:R_0805_2012Metric; symbol Adafruit I2S Audio UDA1334 Bonnet-eagle-import:RESISTOR_0603_NOOUT -> Device:R; LCSC (none) -> C17521
- R26, R27: footprint 0603-NO -> Resistor_SMD:R_0603_1608Metric; symbol Adafruit I2S Audio UDA1334 Bonnet-eagle-import:RESISTOR_0603_NOOUT -> Device:R; LCSC (none) -> C22775
- U7: footprint SOT23-5 -> Package_TO_SOT_SMD:SOT-23-5_HandSoldering
Connections:
- net AGND: now also J8.S; no longer J8.G
- net GPIO16: now also Q4.1 (G), R22.1
- net OUTR: now also J8.R; no longer J8.S
- net at R25.2, R27.1: now also C34.2; no longer C34.-
- net at U8.14 (VOUTL): now also C33.1; no longer C33.+
- net at U8.16 (VOUTR): now also C34.1; no longer C34.+
- net at R24.2, R26.1: now also C33.2; no longer C33.-
- no-connect marks 0 -> 1

Commit message: Everything routed, DRC ok
Connections:
- net GPIO16 is gone; now on net MUTE: Q4.1 (G), R22.1
- net MUTE: no longer Q4.3 (D), R23.2, U8.8 (MUTE)
- net VDD renamed VDDA
- new net: Q4.3 (D), R23.2, U8.8 (MUTE)
Changed lines of the file:
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@@
     (effects (font (size 1.016 1.016)) (justify right bottom))
-  )
-  (label "MUTE" (at 71.755 99.06 0)
-    (effects (font (size 1.5113 1.5113)) (justify left bottom))
   )
   (label "VDDA" (at 84.455 33.02 180)
     (effects (font (size 1.27 1.27)) (justify right bottom))
-  )
-  (label "VDD" (at 84.455 40.64 180)
-    (effects (font (size 1.016 1.016)) (justify right bottom))
   )
   (label "AGND" (at 92.075 66.04 180)
@@
     (effects (font (size 1.016 1.016)) (justify right bottom))
   )
-  (label "OUTL" (at 155.575 63.5 0)
-    (effects (font (size 1.5113 1.5113)) (justify left bottom))
+  (label "OUTL" (at 160.655 63.5 180)
+    (effects (font (size 1.5113 1.5113)) (justify right bottom))
   )
-  (label "OUTR" (at 156.845 83.82 0)
-    (effects (font (size 1.5113 1.5113)) (justify left bottom))
+  (label "OUTR" (at 163.195 83.82 180)
+    (effects (font (size 1.5113 1.5113)) (justify right bottom))
   )
   (label "OUTL" (at 191.77 66.04 0)
@@
     (effects (font (size 1.5113 1.5113)) (justify left bottom))
   )
-  (hierarchical_label "GPIO16" (shape input) (at 31.115 86.36 180)
+  (hierarchical_label "MUTE" (shape input) (at 31.115 86.36 180)
     (effects (font (size 1.27 1.27)) (justify right))
   )
