File: CarPiPowerHat/input_pin_protect.kicad_sch (KiCad schematic)
At the start: 6 parts

Commit message: added connectors
Parts:
- renumbered C22 to C23, D7 to D11, D8 to D12, D9 to D13, D10 to D14, FB2 to FB3
Changed lines of the file:
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@@
   (symbol (lib_id "Device:D_TVS") (at 138.43 86.36 90)
     (in_bom yes) (on_board yes)
-    (property "Reference" "D7" (id 0) (at 140.97 85.09 90)
+    (property "Reference" "D11" (id 0) (at 140.97 85.09 90)
       (effects (font (size 1.27 1.27)) (justify right))
     )
@@
   (symbol (lib_id "Device:D_Schottky") (at 149.86 74.93 270)
     (in_bom yes) (on_board yes)
-    (property "Reference" "D8" (id 0) (at 152.4 73.66 90)
+    (property "Reference" "D12" (id 0) (at 152.4 73.66 90)
       (effects (font (size 1.27 1.27)) (justify left))
     )
@@
   (symbol (lib_id "Device:D_Schottky") (at 149.86 86.36 270)
     (in_bom yes) (on_board yes)
-    (property "Reference" "D9" (id 0) (at 152.4 85.09 90)
+    (property "Reference" "D13" (id 0) (at 152.4 85.09 90)
       (effects (font (size 1.27 1.27)) (justify left))
     )
@@
   (symbol (lib_id "Device:D") (at 165.1 80.01 180)
     (in_bom yes) (on_board yes)
-    (property "Reference" "D10" (id 0) (at 165.1 73.66 0))
+    (property "Reference" "D14" (id 0) (at 165.1 73.66 0))
     (property "Value" "D" (id 1) (at 165.1 76.2 0))
     (property "Footprint" "" (id 2) (at 165.1 80.01 0)
@@
   (symbol (lib_id "Device:C") (at 129.54 86.36 0)
     (in_bom yes) (on_board yes)
-    (property "Reference" "C22" (id 0) (at 133.35 85.09 0)
+    (property "Reference" "C23" (id 0) (at 133.35 85.09 0)
       (effects (font (size 1.27 1.27)) (justify left))
     )
@@
   (symbol (lib_id "Device:FerriteBead") (at 120.65 80.01 90)
     (in_bom yes) (on_board yes)
-    (property "Reference" "FB2" (id 0) (at 120.65 72.39 90))
+    (property "Reference" "FB3" (id 0) (at 120.65 72.39 90))
     (property "Value" "FerriteBead" (id 1) (at 120.65 74.93 90))
     (property "Footprint" "" (id 2) (at 120.65 81.788 90)

Commit message: doing some traces
Parts:
- added R21: 200, Resistor_SMD:R_0402_1005Metric, symbol Device:R
- C23: value C -> 10u; footprint (none) -> Resistor_SMD:R_0603_1608Metric
- D12: footprint (none) -> Diode_SMD:D_SOD-123; LCSC (none) -> C8598
- D13: footprint (none) -> Diode_SMD:D_SOD-123
- D14: footprint (none) -> Diode_SMD:D_SOD-123F; LCSC (none) -> C64898
- FB3: footprint (none) -> Resistor_SMD:R_0805_2012Metric
Connections:
- net at C23.1, D11.2 (A2), D12.2 (A)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: now also R21.1; no longer FB3.2
- new net: FB3.2, R21.2
Other:
- moved on the sheet: FB3
Changed lines of the file:
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@@
   (junction (at 138.43 93.98) (diameter 1.016) (color 0 0 0 0))
   (junction (at 149.86 80.01) (diameter 1.016) (color 0 0 0 0))
-  (wire (pts (xy 113.03 80.01) (xy 116.84 80.01))
+  (wire (pts (xy 104.14 80.01) (xy 107.95 80.01))
     (stroke (width 0) (type solid) (color 0 0 0 0))
   )
-  (wire (pts (xy 113.665 64.77) (xy 149.86 64.77))
+  (wire (pts (xy 104.775 64.77) (xy 149.86 64.77))
     (stroke (width 0) (type solid) (color 0 0 0 0))
   )
-  (wire (pts (xy 124.46 80.01) (xy 129.54 80.01))
+  (wire (pts (xy 115.57 80.01) (xy 118.11 80.01))
+    (stroke (width 0) (type solid) (color 0 0 0 0))
+  )
+  (wire (pts (xy 125.73 80.01) (xy 129.54 80.01))
     (stroke (width 0) (type solid) (color 0 0 0 0))
   )
@@
     (stroke (width 0) (type solid) (color 0 0 0 0))
   )
-  (hierarchical_label "IN" (shape input) (at 113.03 80.01 180)
+  (hierarchical_label "IN" (shape input) (at 104.14 80.01 180)
     (effects (font (size 1.27 1.27)) (justify right))
   )
-  (hierarchical_label "+3.3v" (shape input) (at 113.665 64.77 180)
+  (hierarchical_label "+3.3v" (shape input) (at 104.775 64.77 180)
     (effects (font (size 1.27 1.27)) (justify right))
   )
@@
   (hierarchical_label "OUT" (shape output) (at 173.99 80.01 0)
     (effects (font (size 1.27 1.27)) (justify left))
+  )
+  (symbol (lib_id "Device:R") (at 121.92 80.01 270)
+    (in_bom yes) (on_board yes)
+    (property "Reference" "R21" (id 0) (at 121.92 74.93 90))
+    (property "Value" "200" (id 1) (at 121.92 77.47 90))
+    (property "Footprint" "Resistor_SMD:R_0402_1005Metric" (id 2) (at 121.92 78.232 90)
+      (effects (font (size 1.27 1.27)) hide)
+    )
+    (property "Datasheet" "~" (id 3) (at 121.92 80.01 0)
+      (effects (font (size 1.27 1.27)) hide)
+    )
+    (pin "1")
+    (pin "2")
   )
   (symbol (lib_id "Device:D_TVS") (at 138.43 86.36 90)
@@
       (effects (font (size 1.27 1.27)) (justify left))
     )
-    (property "Footprint" "" (id 2) (at 149.86 74.93 0)
+    (property "Footprint" "Diode_SMD:D_SOD-123" (id 2) (at 149.86 74.93 0)
       (effects (font (size 1.27 1.27)) hide)
     )
     (property "Datasheet" "~" (id 3) (at 149.86 74.93 0)
+      (effects (font (size 1.27 1.27)) hide)
+    )
+    (property "LCSC" "C8598" (id 4) (at 149.86 74.93 90)
       (effects (font (size 1.27 1.27)) hide)
     )
@@
       (effects (font (size 1.27 1.27)) (justify left))
     )
-    (property "Footprint" "" (id 2) (at 149.86 86.36 0)
+    (property "Footprint" "Diode_SMD:D_SOD-123" (id 2) (at 149.86 86.36 0)
       (effects (font (size 1.27 1.27)) hide)
     )
@@
     (property "Reference" "D14" (id 0) (at 165.1 73.66 0))
     (property "Value" "D" (id 1) (at 165.1 76.2 0))
-    (property "Footprint" "" (id 2) (at 165.1 80.01 0)
+    (property "Footprint" "Diode_SMD:D_SOD-123F" (id 2) (at 165.1 80.01 0)
       (effects (font (size 1.27 1.27)) hide)
     )
     (property "Datasheet" "~" (id 3) (at 165.1 80.01 0)
+      (effects (font (size 1.27 1.27)) hide)
+    )
+    (property "LCSC" "C64898" (id 4) (at 165.1 80.01 0)
       (effects (font (size 1.27 1.27)) hide)
     )
@@
       (effects (font (size 1.27 1.27)) (justify left))
     )
-    (property "Value" "C" (id 1) (at 133.35 87.63 0)
+    (property "Value" "10u" (id 1) (at 133.35 87.63 0)
       (effects (font (size 1.27 1.27)) (justify left))
     )
-    (property "Footprint" "" (id 2) (at 130.5052 90.17 0)
+    (property "Footprint" "Resistor_SMD:R_0603_1608Metric" (id 2) (at 130.5052 90.17 0)
       (effects (font (size 1.27 1.27)) hide)
     )
@@
     (pin "2")
   )
-  (symbol (lib_id "Device:FerriteBead") (at 120.65 80.01 90)
+  (symbol (lib_id "Device:FerriteBead") (at 111.76 80.01 90)
     (in_bom yes) (on_board yes)
-    (property "Reference" "FB3" (id 0) (at 120.65 72.39 90))
-    (property "Value" "FerriteBead" (id 1) (at 120.65 74.93 90))
-    (property "Footprint" "" (id 2) (at 120.65 81.788 90)
+    (property "Reference" "FB3" (id 0) (at 111.76 72.39 90))
+    (property "Value" "FerriteBead" (id 1) (at 111.76 74.93 90))
+    (property "Footprint" "Resistor_SMD:R_0805_2012Metric" (id 2) (at 111.76 81.788 90)
       (effects (font (size 1.27 1.27)) hide)
     )
-    (property "Datasheet" "~" (id 3) (at 120.65 80.01 0)
+    (property "Datasheet" "~" (id 3) (at 111.76 80.01 0)
       (effects (font (size 1.27 1.27)) hide)
     )

Commit message: Everything routed, DRC ok
Parts:
- D11: footprint (none) -> Diode_SMD:D_0603_1608Metric
Changed lines of the file:
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@@
       (effects (font (size 1.27 1.27)) (justify right))
     )
-    (property "Footprint" "" (id 2) (at 138.43 86.36 0)
+    (property "Footprint" "Diode_SMD:D_0603_1608Metric" (id 2) (at 138.43 86.36 0)
       (effects (font (size 1.27 1.27)) hide)
     )
