File: CarPiPowerHat/input_pin_protect.kicad_sch (KiCad schematic)
At the start: 5 parts

Commit message: Some bugfixing, added cam.py script
Changed lines of the file:
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@@
-(kicad_sch (version 20210621) (generator eeschema)
+(kicad_sch (version 20211123) (generator eeschema)
   (paper "A4")
-  (junction (at 120.65 80.01) (diameter 1.016) (color 0 0 0 0))
-  (junction (at 129.54 80.01) (diameter 1.016) (color 0 0 0 0))
-  (junction (at 129.54 93.98) (diameter 1.016) (color 0 0 0 0))
-  (junction (at 143.51 80.01) (diameter 1.016) (color 0 0 0 0))
-  (junction (at 143.51 93.98) (diameter 1.016) (color 0 0 0 0))
-  (junction (at 167.005 80.01) (diameter 1.016) (color 0 0 0 0))
+  (junction (at 129.54 93.98) (diameter 1.016) (color 0 0 0 0)
+  )
+  (junction (at 129.54 80.01) (diameter 1.016) (color 0 0 0 0)
+  )
+  (junction (at 160.02 80.01) (diameter 0) (color 0 0 0 0)
+  )
+  (junction (at 143.51 80.01) (diameter 1.016) (color 0 0 0 0)
+  )
+  (junction (at 120.65 80.01) (diameter 1.016) (color 0 0 0 0)
+  )
+  (junction (at 143.51 93.98) (diameter 1.016) (color 0 0 0 0)
+  )
+  (wire (pts (xy 129.54 80.01) (xy 129.54 82.55))
+    (stroke (width 0) (type solid) (color 0 0 0 0))
+  )
+  (wire (pts (xy 143.51 93.98) (xy 143.51 97.155))
+    (stroke (width 0) (type solid) (color 0 0 0 0))
+  )
+  (wire (pts (xy 129.54 80.01) (xy 143.51 80.01))
+    (stroke (width 0) (type solid) (color 0 0 0 0))
+  )
+  (wire (pts (xy 160.02 80.01) (xy 179.07 80.01))
+    (stroke (width 0) (type solid) (color 0 0 0 0))
+  )
+  (wire (pts (xy 154.94 93.98) (xy 143.51 93.98))
+    (stroke (width 0) (type solid) (color 0 0 0 0))
+  )
   (wire (pts (xy 104.14 80.01) (xy 109.22 80.01))
+    (stroke (width 0) (type solid) (color 0 0 0 0))
+  )
+  (wire (pts (xy 116.84 80.01) (xy 120.65 80.01))
+    (stroke (width 0) (type solid) (color 0 0 0 0))
+  )
+  (wire (pts (xy 120.65 80.01) (xy 129.54 80.01))
+    (stroke (width 0) (type solid) (color 0 0 0 0))
+  )
+  (wire (pts (xy 143.51 97.155) (xy 147.955 97.155))
+    (stroke (width 0) (type solid) (color 0 0 0 0))
+  )
+  (wire (pts (xy 143.51 82.55) (xy 143.51 80.01))
+    (stroke (width 0) (type solid) (color 0 0 0 0))
+  )
+  (wire (pts (xy 143.51 80.01) (xy 160.02 80.01))
+    (stroke (width 0) (type solid) (color 0 0 0 0))
+  )
+  (wire (pts (xy 154.94 87.63) (xy 154.94 93.98))
+    (stroke (width 0) (type solid) (color 0 0 0 0))
+  )
+  (wire (pts (xy 120.65 80.01) (xy 120.65 82.55))
+    (stroke (width 0) (type solid) (color 0 0 0 0))
+  )
+  (wire (pts (xy 143.51 93.98) (xy 143.51 90.17))
+    (stroke (width 0) (type solid) (color 0 0 0 0))
+  )
+  (wire (pts (xy 129.54 90.17) (xy 129.54 93.98))
     (stroke (width 0) (type solid) (color 0 0 0 0))
   )
@@
     (stroke (width 0) (type solid) (color 0 0 0 0))
   )
-  (wire (pts (xy 116.84 80.01) (xy 120.65 80.01))
-    (stroke (width 0) (type solid) (color 0 0 0 0))
-  )
-  (wire (pts (xy 120.65 80.01) (xy 120.65 82.55))
-    (stroke (width 0) (type solid) (color 0 0 0 0))
-  )
-  (wire (pts (xy 120.65 80.01) (xy 129.54 80.01))
+  (wire (pts (xy 154.94 64.77) (xy 154.94 72.39))
     (stroke (width 0) (type solid) (color 0 0 0 0))
   )
@@
     (stroke (width 0) (type solid) (color 0 0 0 0))
   )
-  (wire (pts (xy 129.54 80.01) (xy 129.54 82.55))
-    (stroke (width 0) (type solid) (color 0 0 0 0))
-  )
-  (wire (pts (xy 129.54 80.01) (xy 143.51 80.01))
-    (stroke (width 0) (type solid) (color 0 0 0 0))
-  )
-  (wire (pts (xy 129.54 90.17) (xy 129.54 93.98))
-    (stroke (width 0) (type solid) (color 0 0 0 0))
-  )
   (wire (pts (xy 129.54 93.98) (xy 143.51 93.98))
     (stroke (width 0) (type solid) (color 0 0 0 0))
   )
-  (wire (pts (xy 143.51 71.12) (xy 167.005 71.12))
-    (stroke (width 0) (type solid) (color 0 0 0 0))
+  (hierarchical_label "OUT" (shape output) (at 179.07 80.01 0)
+    (effects (font (size 1.27 1.27)) (justify left))
   )
-  (wire (pts (xy 143.51 80.01) (xy 143.51 71.12))
-    (stroke (width 0) (type solid) (color 0 0 0 0))
-  )
-  (wire (pts (xy 143.51 82.55) (xy 143.51 80.01))
-    (stroke (width 0) (type solid) (color 0 0 0 0))
-  )
-  (wire (pts (xy 143.51 93.98) (xy 143.51 90.17))
-    (stroke (width 0) (type solid) (color 0 0 0 0))
-  )
-  (wire (pts (xy 143.51 93.98) (xy 143.51 97.155))
-    (stroke (width 0) (type solid) (color 0 0 0 0))
-  )
-  (wire (pts (xy 143.51 97.155) (xy 147.955 97.155))
-    (stroke (width 0) (type solid) (color 0 0 0 0))
-  )
-  (wire (pts (xy 154.94 64.77) (xy 154.94 72.39))
-    (stroke (width 0) (type solid) (color 0 0 0 0))
-  )
-  (wire (pts (xy 154.94 87.63) (xy 154.94 93.98))
-    (stroke (width 0) (type solid) (color 0 0 0 0))
-  )
-  (wire (pts (xy 154.94 93.98) (xy 143.51 93.98))
-    (stroke (width 0) (type solid) (color 0 0 0 0))
-  )
-  (wire (pts (xy 160.02 80.01) (xy 167.005 80.01))
-    (stroke (width 0) (type solid) (color 0 0 0 0))
-  )
-  (wire (pts (xy 167.005 71.12) (xy 167.005 80.01))
-    (stroke (width 0) (type solid) (color 0 0 0 0))
-  )
-  (wire (pts (xy 167.005 80.01) (xy 179.07 80.01))
-    (stroke (width 0) (type solid) (color 0 0 0 0))
+  (hierarchical_label "+3.3v" (shape input) (at 104.775 64.77 180)
+    (effects (font (size 1.27 1.27)) (justify right))
   )
   (hierarchical_label "IN" (shape input) (at 104.14 80.01 180)
     (effects (font (size 1.27 1.27)) (justify right))
   )
-  (hierarchical_label "+3.3v" (shape input) (at 104.775 64.77 180)
-    (effects (font (size 1.27 1.27)) (justify right))
-  )
   (hierarchical_label "GND" (shape output) (at 147.955 97.155 0)
-    (effects (font (size 1.27 1.27)) (justify left))
-  )
-  (hierarchical_label "OUT" (shape output) (at 179.07 80.01 0)
     (effects (font (size 1.27 1.27)) (justify left))
   )
@@
     (pin "2")
   )
-  (symbol (lib_id "Device:R") (at 120.65 86.36 0)
+  (symbol (lib_id "Diode:BAT54S") (at 154.94 80.01 90)
     (in_bom yes) (on_board yes)
-    (property "Reference" "R28" (id 0) (at 115.57 86.36 90))
-    (property "Value" "1M" (id 1) (at 118.11 86.36 90))
-    (property "Footprint" "Resistor_SMD:R_0805_2012Metric_Pad1.20x1.40mm_HandSolder" (id 2) (at 118.872 86.36 90)
+    (property "Reference" "D5" (id 0) (at 163.83 78.7399 90)
+      (effects (font (size 1.27 1.27)) (justify left))
+    )
+    (property "Value" "BAT54S" (id 1) (at 163.83 81.2799 90)
+      (effects (font (size 1.27 1.27)) (justify left))
+    )
+    (property "Footprint" "Package_TO_SOT_SMD:SOT-23" (id 2) (at 151.765 78.105 0)
+      (effects (font (size 1.27 1.27)) (justify left) hide)
+    )
+    (property "Datasheet" "https://www.diodes.com/assets/Datasheets/ds11005.pdf" (id 3) (at 154.94 83.058 0)
       (effects (font (size 1.27 1.27)) hide)
     )
-    (property "Datasheet" "~" (id 3) (at 120.65 86.36 0)
-      (effects (font (size 1.27 1.27)) hide)
-    )
-    (property "LCSC" "C17514" (id 4) (at 120.65 86.36 0)
+    (property "LCSC" "C408389" (id 4) (at 154.94 80.01 0)
       (effects (font (size 1.27 1.27)) hide)
     )
     (pin "1")
     (pin "2")
+    (pin "3")
   )
   (symbol (lib_id "Device:D_TVS") (at 143.51 86.36 90)
@@
     (pin "2")
   )
-  (symbol (lib_id "Diode:BAT54S") (at 154.94 80.01 90)
+  (symbol (lib_id "Device:R") (at 120.65 86.36 0)
     (in_bom yes) (on_board yes)
-    (property "Reference" "D5" (id 0) (at 163.83 78.7399 90)
-      (effects (font (size 1.27 1.27)) (justify left))
-    )
-    (property "Value" "BAT54S" (id 1) (at 163.83 81.2799 90)
-      (effects (font (size 1.27 1.27)) (justify left))
-    )
-    (property "Footprint" "Package_TO_SOT_SMD:SOT-23" (id 2) (at 151.765 78.105 0)
-      (effects (font (size 1.27 1.27)) (justify left) hide)
-    )
-    (property "Datasheet" "https://www.diodes.com/assets/Datasheets/ds11005.pdf" (id 3) (at 154.94 83.058 0)
+    (property "Reference" "R28" (id 0) (at 115.57 86.36 90))
+    (property "Value" "1M" (id 1) (at 118.11 86.36 90))
+    (property "Footprint" "Resistor_SMD:R_0805_2012Metric_Pad1.20x1.40mm_HandSolder" (id 2) (at 118.872 86.36 90)
       (effects (font (size 1.27 1.27)) hide)
     )
-    (property "LCSC" "C408389" (id 4) (at 154.94 80.01 0)
+    (property "Datasheet" "~" (id 3) (at 120.65 86.36 0)
+      (effects (font (size 1.27 1.27)) hide)
+    )
+    (property "LCSC" "C17514" (id 4) (at 120.65 86.36 0)
       (effects (font (size 1.27 1.27)) hide)
     )
     (pin "1")
     (pin "2")
-    (pin "3")
   )
 )
