File: CarPiPowerHat/power_control.kicad_sch (KiCad schematic)
At the start: 16 parts, among them U3 LM3480-5.0, U4 ATtiny45V-10X

Commit message: doing some traces
Parts:
- D2: footprint (none) -> LED_SMD:LED_0603_1608Metric
- D6: footprint (none) -> Package_TO_SOT_SMD:SOT-23
Changed lines of the file:
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@@
       (effects (font (size 1.27 1.27)) hide)
     )
-    (property "Datasheet" "" (id 3) (at 85.725 40.005 0)
+    (property "Datasheet" "~" (id 3) (at 85.725 40.005 0)
       (effects (font (size 1.27 1.27)) hide)
     )
@@
       (effects (font (size 1.27 1.27)) hide)
     )
-    (property "Datasheet" "https://fscdn.rohm.com/en/products/databook/datasheet/passive/resistor/chip_resistor/mcr-e.pdf" (id 3) (at 137.795 50.165 0)
+    (property "Datasheet" "~" (id 3) (at 137.795 50.165 0)
       (effects (font (size 1.27 1.27)) hide)
     )
@@
       (effects (font (size 1.27 1.27)) hide)
     )
-    (property "Datasheet" "https://fscdn.rohm.com/en/products/databook/datasheet/passive/resistor/chip_resistor/mcr-e.pdf" (id 3) (at 146.685 41.275 0)
+    (property "Datasheet" "~" (id 3) (at 146.685 41.275 0)
       (effects (font (size 1.27 1.27)) hide)
     )
@@
       (effects (font (size 1.27 1.27)) hide)
     )
-    (property "Datasheet" "https://fscdn.rohm.com/en/products/databook/datasheet/passive/resistor/chip_resistor/mcr-e.pdf" (id 3) (at 152.4 72.39 0)
+    (property "Datasheet" "~" (id 3) (at 152.4 72.39 0)
       (effects (font (size 1.27 1.27)) hide)
     )
@@
       (effects (font (size 1.27 1.27)) hide)
     )
-    (property "Datasheet" "https://fscdn.rohm.com/en/products/databook/datasheet/passive/resistor/chip_resistor/mcr-e.pdf" (id 3) (at 164.465 39.37 0)
+    (property "Datasheet" "~" (id 3) (at 164.465 39.37 0)
       (effects (font (size 1.27 1.27)) hide)
     )
@@
       (effects (font (size 1.27 1.27)) hide)
     )
-    (property "Datasheet" "https://fscdn.rohm.com/en/products/databook/datasheet/passive/resistor/chip_resistor/mcr-e.pdf" (id 3) (at 170.18 68.58 0)
+    (property "Datasheet" "~" (id 3) (at 170.18 68.58 0)
       (effects (font (size 1.27 1.27)) hide)
     )
@@
       (effects (font (size 1.27 1.27)) hide)
     )
-    (property "Datasheet" "https://fscdn.rohm.com/en/products/databook/datasheet/passive/resistor/chip_resistor/mcr-e.pdf" (id 3) (at 170.18 78.74 0)
+    (property "Datasheet" "~" (id 3) (at 170.18 78.74 0)
       (effects (font (size 1.27 1.27)) hide)
     )
@@
       (effects (font (size 1.27 1.27)) hide)
     )
-    (property "Datasheet" "https://fscdn.rohm.com/en/products/databook/datasheet/passive/resistor/chip_resistor/mcr-e.pdf" (id 3) (at 187.96 68.58 0)
+    (property "Datasheet" "~" (id 3) (at 187.96 68.58 0)
       (effects (font (size 1.27 1.27)) hide)
     )
@@
       (effects (font (size 1.27 1.27)) (justify right))
     )
-    (property "Footprint" "" (id 2) (at 164.465 47.625 0)
+    (property "Footprint" "LED_SMD:LED_0603_1608Metric" (id 2) (at 164.465 47.625 0)
       (effects (font (size 1.27 1.27)) hide)
     )
@@
       (effects (font (size 1.27 1.27)) hide)
     )
-    (property "Datasheet" "https://search.murata.co.jp/Ceramy/image/img/A01X/G101/ENG/GRM155R71C104KA88-01.pdf" (id 3) (at 55.245 51.435 0)
+    (property "Datasheet" "~" (id 3) (at 55.245 51.435 0)
       (effects (font (size 1.27 1.27)) hide)
     )
@@
       (effects (font (size 1.27 1.27)) hide)
     )
-    (property "Datasheet" "https://search.murata.co.jp/Ceramy/image/img/A01X/G101/ENG/GRM155R71C104KA88-01.pdf" (id 3) (at 80.645 51.435 0)
+    (property "Datasheet" "~" (id 3) (at 80.645 51.435 0)
       (effects (font (size 1.27 1.27)) hide)
     )
@@
     (property "Reference" "D6" (id 0) (at 100.965 24.765 0))
     (property "Value" "D_Dual_CommonCathode_AAK_Parallel" (id 1) (at 100.965 27.305 0))
-    (property "Footprint" "" (id 2) (at 101.6 33.655 0)
-      (effects (font (size 1.27 1.27)) hide)
-    )
+    (property "Footprint" "Package_TO_SOT_SMD:SOT-23" (id 2) (at 101.6 33.655 0)
+      (effects (font (size 1.27 1.27)) hide)
+    )

Commit message: doing some traces
Parts:
- added D1: LED, LED_SMD:LED_0603_1608Metric, symbol Device:LED
- added R11: 130, Resistor_SMD:R_0603_1608Metric, symbol Device:R
- added R28: 10K 1%, Resistor_SMD:R_0603_1608Metric, symbol Device:R
- added TP6, TP7: TestPoint, TestPoint:TestPoint_Pad_2.0x2.0mm, symbol Connector:TestPoint
- C20, C21: LCSC (none) -> C1525
- D2: LCSC (none) -> C72041
- D5: footprint (none) -> Diode_SMD:D_0603_1608Metric_Pad1.05x0.95mm_HandSolder
- D6: LCSC (none) -> C68978
- R13, R14, R15, R16, R17: footprint Resistor_SMD:R_0402_1005Metric -> Resistor_SMD:R_0603_1608Metric; LCSC (none) -> C25804
- R18: value 320 1% -> 200 1%; LCSC (none) -> C25087
- R19: footprint Resistor_SMD:R_0402_1005Metric -> Resistor_SMD:R_0603_1608Metric; LCSC (none) -> C22978
- U3: LCSC (none) -> C129960
Connections:
- net GND: now also R11.2, R28.2
- net IGN: now also C20.1, D5.2 (A2), F2.2, U3.2 (VI)
- net PSU_EN: now also U4.2 (XTAL1/PB3); no longer U4.5 (AREF/PB0)
- net PWR_SENSE_OUT: now also D1.2 (A)
- net at R19.1, U4.7 (PB2): now also R28.1
- net VO: now reaches C21.1, D6.2 (K), R19.2, TP4.1, U3.1 (VO)
- net at R14.1: now also U4.5 (AREF/PB0); no longer U4.2 (XTAL1/PB3)
- net at D2.2 (A), R18.2: now also TP6.1
- net VCC: now reaches D6.3 (A), R17.1, U4.8 (VCC)
- new net: D1.1 (K), R11.1, TP7.1
Other:
- moved on the sheet: R16

Commit message: Everything routed, DRC ok
Connections:
- net IGN: no longer C20.1, D5.2 (A2), F2.2, U3.2 (VI)
- net P5V_HAT renamed +5v
- new net: C20.1, D5.2 (A2), F2.2, U3.2 (VI)
Changed lines of the file:
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@@
-    (effects (font (size 1.27 1.27)) (justify right bottom))
-  )
-  (label "IGN" (at 51.435 43.815 180)
     (effects (font (size 1.27 1.27)) (justify right bottom))
   )
@@
     )
   )
-  (hierarchical_label "P5V_HAT" (shape input) (at 26.67 31.115 180)
+  (hierarchical_label "+5v" (shape input) (at 26.67 31.115 180)
     (effects (font (size 1.27 1.27)) (justify right))
   )
