File: CarPiPowerHat/power_control.kicad_sch (KiCad schematic)
At the start: 21 parts, among them J11 Conn_01x06_Male, U2 ATtiny45V-20SU, U7 LM3480-5.0

Commit message: Finalizing, checking parts
Might be ready for production
Parts:
- D10: value LED Red -> LED Green
- D6: LCSC C181200 -> C37704
- D9: value LED Green -> LED Blue; LCSC C72041 -> C72041
Changed lines of the file:
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@@
       (effects (font (size 1.27 1.27)) (justify right))
     )
-    (property "Value" "LED Green" (id 1) (at 177.8 49.53 90)
+    (property "Value" "LED Blue" (id 1) (at 177.8 49.53 90)
       (effects (font (size 1.27 1.27)) (justify right))
     )
@@
       (effects (font (size 1.27 1.27)) hide)
     )
-    (property "LCSC" " C72041" (id 4) (at 174.625 47.625 90)
+    (property "LCSC" "C72041" (id 4) (at 174.625 47.625 90)
       (effects (font (size 1.27 1.27)) hide)
     )
@@
       (effects (font (size 1.27 1.27)) (justify right))
     )
-    (property "Value" "LED Red" (id 1) (at 194.945 38.1 90)
+    (property "Value" "LED Green" (id 1) (at 194.945 38.1 90)
       (effects (font (size 1.27 1.27)) (justify right))
     )
@@
       (effects (font (size 1.27 1.27)) hide)
     )
-    (property "LCSC" "C181200" (id 9) (at 100.33 33.655 90)
+    (property "LCSC" "C37704" (id 9) (at 100.33 33.655 90)
       (effects (font (size 1.27 1.27)) hide)
     )
