File: CarPiPowerHat/psu.kicad_sch (KiCad schematic)
At the start: 38 parts, among them Q1 DMMT5401, Q2 DMG2305UX, Q3 DMP3013SFV-7, U1 AP64501SP-13

Commit message: doing some traces
Parts:
- added C25, C26: 100n, Capacitor_SMD:C_0402_1005Metric, symbol Device:C
- added J5: USB_A, Connector_USB:USB_A_Wuerth_614004134726_Horizontal, symbol Connector:USB_A
- added U6: RT9742SNGV, Package_TO_SOT_SMD:SOT-23, symbol CM4IO:RT9742SNGV
- C19: symbol Device:CP -> Device:C_Polarized
- Q1: footprint SOT-26 -> project_footprints:SOT26; symbol raspberrypi_hat:DMMT5401 -> CarPiPowerHat:DMMT5401
- Q2: symbol raspberrypi_hat:DMG2305UX -> CarPiPowerHat:DMG2305UX
- R1, R4: footprint Resistor_SMD:R_0603_1608Metric_Pad0.84x1.00mm_HandSolder -> Resistor_SMD:R_0402_1005Metric_Pad0.72x0.64mm_HandSolder
Connections:
- net +5v: now also C25.1, U6.1 (IN)
- net GND: now also C25.2, C26.2, J5.4 (GND), J5.5 (Shield), U6.3 (GND)
- new net USB_5v: C26.1, J5.1 (VBUS), U6.2 (OUT)
- no-connect marks 0 -> 2

Commit message: doing some traces
Parts:
- C1, C2, C3, C5, C6, C7: LCSC (none) -> C469541
- C13: footprint Capacitor_SMD:C_0402_1005Metric -> Capacitor_SMD:C_0603_1608Metric; LCSC (none) -> C30615
- C15, C16, C17, C18: LCSC (none) -> C15850
- C19: LCSC (none) -> C16133
- C8, C9: LCSC (none) -> C1525
- R10: LCSC (none) -> C25752
- R12: LCSC (none) -> C25879
- R9: LCSC (none) -> C25765
Connections:
- net +5v: no longer C25.1, U6.1 (IN)
- net P5V: now also C25.1, U6.1 (IN)
Changed lines of the file:
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@@
     (effects (font (size 1.524 1.524)) (justify left bottom))
+  )
+  (label "P5V" (at 230.505 59.69 180)
+    (effects (font (size 1.524 1.524)) (justify right bottom))
   )
   (label "P5V" (at 236.22 98.425 180)
@@
   (hierarchical_label "GND" (shape output) (at 226.695 123.19 0)
     (effects (font (size 1.27 1.27)) (justify left))
-  )
-  (hierarchical_label "+5v" (shape input) (at 230.505 59.69 180)
-    (effects (font (size 1.27 1.27)) (justify right))
   )
   (symbol (lib_id "Connector:TestPoint") (at 125.73 36.068 0) (unit 1)
@@
       (effects (font (size 1.27 1.27)) hide)
     )
+    (property "LCSC" "C25765" (id 9) (at 144.78 122.682 0)
+      (effects (font (size 1.27 1.27)) hide)
+    )
     (pin "1")
     (pin "2")
@@
       (effects (font (size 1.27 1.27)) hide)
     )
+    (property "LCSC" "C25752" (id 9) (at 154.94 109.982 0)
+      (effects (font (size 1.27 1.27)) hide)
+    )
     (pin "1")
     (pin "2")
@@
     )
     (property "Field8" "120889581" (id 9) (at 154.94 129.032 0)
+      (effects (font (size 1.27 1.27)) hide)
+    )
+    (property "LCSC" "C25879" (id 10) (at 154.94 129.032 0)
       (effects (font (size 1.27 1.27)) hide)
     )
@@
       (effects (font (size 1.27 1.27)) hide)
     )
+    (property "LCSC" "C469541" (id 10) (at 41.275 116.205 0)
+      (effects (font (size 1.27 1.27)) hide)
+    )
     (pin "1")
     (pin "2")
@@
       (effects (font (size 1.27 1.27)) hide)
     )
+    (property "LCSC" "C469541" (id 10) (at 52.07 116.205 0)
+      (effects (font (size 1.27 1.27)) hide)
+    )
     (pin "1")
     (pin "2")
@@
       (effects (font (size 1.27 1.27)) hide)
     )
+    (property "LCSC" "C469541" (id 10) (at 62.865 116.205 0)
+      (effects (font (size 1.27 1.27)) hide)
+    )
     (pin "1")
     (pin "2")
@@
       (effects (font (size 1.27 1.27)) hide)
     )
+    (property "LCSC" "C469541" (id 10) (at 73.025 116.205 0)
+      (effects (font (size 1.27 1.27)) hide)
+    )
     (pin "1")
     (pin "2")
@@
       (effects (font (size 1.27 1.27)) hide)
     )
+    (property "LCSC" "C469541" (id 10) (at 83.82 116.205 0)
+      (effects (font (size 1.27 1.27)) hide)
+    )
     (pin "1")
     (pin "2")
@@
       (effects (font (size 1.27 1.27)) hide)
     )
+    (property "LCSC" "C469541" (id 10) (at 95.25 116.205 0)
+      (effects (font (size 1.27 1.27)) hide)
+    )
     (pin "1")
     (pin "2")
@@
       (effects (font (size 1.27 1.27)) hide)
     )
+    (property "LCSC" "C1525" (id 10) (at 104.775 104.267 0)
+      (effects (font (size 1.27 1.27)) hide)
+    )
     (pin "1")
     (pin "2")
@@
       (effects (font (size 1.27 1.27)) hide)
     )
+    (property "LCSC" "C1525" (id 10) (at 108.585 126.492 0)
+      (effects (font (size 1.27 1.27)) hide)
+    )
     (pin "1")
     (pin "2")
@@
       (effects (font (size 1.27 1.27)) (justify left))
     )
-    (property "Footprint" "Capacitor_SMD:C_0402_1005Metric" (id 2) (at 145.7452 134.112 0)
+    (property "Footprint" "Capacitor_SMD:C_0603_1608Metric" (id 2) (at 145.7452 134.112 0)
       (effects (font (size 1.27 1.27)) hide)
     )
@@
       (effects (font (size 1.27 1.27)) hide)
     )
+    (property "LCSC" "C30615" (id 9) (at 144.78 130.302 0)
+      (effects (font (size 1.27 1.27)) hide)
+    )
     (pin "1")
     (pin "2")
@@
       (effects (font (size 1.27 1.27)) hide)
     )
+    (property "LCSC" "C15850" (id 10) (at 184.15 102.362 0)
+      (effects (font (size 1.27 1.27)) hide)
+    )
     (pin "1")
     (pin "2")
@@
       (effects (font (size 1.27 1.27)) hide)
     )
+    (property "LCSC" "C15850" (id 10) (at 194.31 102.362 0)
+      (effects (font (size 1.27 1.27)) hide)
+    )
     (pin "1")
     (pin "2")
@@
       (effects (font (size 1.27 1.27)) hide)
     )
+    (property "LCSC" "C15850" (id 10) (at 204.47 102.362 0)
+      (effects (font (size 1.27 1.27)) hide)
+    )
     (pin "1")
     (pin "2")
@@
       (effects (font (size 1.27 1.27)) hide)
     )
+    (property "LCSC" "C15850" (id 10) (at 213.36 102.362 0)
+      (effects (font (size 1.27 1.27)) hide)
+    )
     (pin "1")
     (pin "2")
@@
       (effects (font (size 1.27 1.27)) hide)
     )
+    (property "LCSC" "C16133" (id 7) (at 227.457 102.362 0)
+      (effects (font (size 1.27 1.27)) hide)
+    )

Commit message: Everything routed, DRC ok
Parts:
- removed U6: RT9742SNGV, Package_TO_SOT_SMD:SOT-23, symbol CM4IO:RT9742SNGV
- added IC1: AP2331TDSA-7, ap2331:SOT96P240X110-3N, symbol AP2331TDSA-7:AP2331TDSA-7
- added J10: Conn_01x02_Male, Connector_JST:JST_XH_S2B-XH-A_1x02_P2.50mm_Horizontal, symbol Connector:Conn_01x02_Male
- C10, C25, C26, C4: LCSC (none) -> C1525
- C11: LCSC (none) -> C469541
- D4: LCSC (none) -> C268585
- Q1: LCSC (none) -> C154733
- Q2: LCSC (none) -> C144153
- R5: LCSC (none) -> C25879
Connections:
- net +5v: now also J10.2 (Pin_2)
- net GND: now also IC1.1 (GND), J10.1 (Pin_1)
- net P5V: now also IC1.3 (IN)
- net USB_5v: now also IC1.2 (OUT)
Other:
- note added: "SSD Power Out"
- note added: "USB Power Out"
- moved on the sheet: C25, C26, J5
