File: CarPiPowerHat/CarPiPowerHat.kicad_sch (KiCad schematic)
At the start: 8 parts, among them J2 Conn_01x04, J6 Conn_02x03_Counter_Clockwise

Commit message: Finalizing, checking parts
Might be ready for production
Parts:
- J2: footprint Connector_PinHeader_1.00mm:PinHeader_1x04_P1.00mm_Vertical -> Connector_PinHeader_2.00mm:PinHeader_1x04_P2.00mm_Vertical
Changed lines of the file:
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@@
     (property "Reference" "J2" (id 0) (at 45.847 186.69 0))
     (property "Value" "Conn_01x04" (id 1) (at 45.847 189.23 0))
-    (property "Footprint" "Connector_PinHeader_1.00mm:PinHeader_1x04_P1.00mm_Vertical" (id 2) (at 43.815 196.85 0)
+    (property "Footprint" "Connector_PinHeader_2.00mm:PinHeader_1x04_P2.00mm_Vertical" (id 2) (at 43.815 196.85 0)
       (effects (font (size 1.27 1.27)) hide)
     )
@@
     )
     (path "/d7dab0b1-a885-42c4-b558-97d79e73318c/d7f1481a-aaa9-45ad-b805-e8818d9de408"
-      (reference "C38") (unit 1) (value "100uF") (footprint "Capacitor_SMD:C_0603_1608Metric_Pad1.08x0.95mm_HandSolder")
+      (reference "C38") (unit 1) (value "100uF") (footprint "Capacitor_SMD:C_1206_3216Metric_Pad1.33x1.80mm_HandSolder")
     )
     (path "/d7dab0b1-a885-42c4-b558-97d79e73318c/6a588fdd-0512-4cb7-88bc-a8880f02101d"
@@
     )
     (path "/c779e344-5031-4f2d-bf31-77741b3c4be9/9fef9f7d-ce53-455a-b81f-ed54ca115295"
-      (reference "D9") (unit 1) (value "LED Green") (footprint "LED_SMD:LED_0603_1608Metric")
+      (reference "D9") (unit 1) (value "LED Blue") (footprint "LED_SMD:LED_0603_1608Metric")
     )
     (path "/c779e344-5031-4f2d-bf31-77741b3c4be9/4b70c4e6-76ec-4cce-ba57-391430d49c52"
-      (reference "D10") (unit 1) (value "LED Red") (footprint "LED_SMD:LED_0603_1608Metric")
+      (reference "D10") (unit 1) (value "LED Green") (footprint "LED_SMD:LED_0603_1608Metric")
     )
     (path "/c779e344-5031-4f2d-bf31-77741b3c4be9/bf96bf44-e2de-4690-a691-c8b28c5fe37d"
@@
     )
     (path "/696a3b6b-1b33-4b36-bded-7b3fb05e770a/fdabd193-05b7-418b-b423-c7f9635f8ada"
-      (reference "J1") (unit 1) (value "1-84953-5") (footprint "project_footprints:1849535")
+      (reference "J1") (unit 1) (value "1-84953-5") (footprint "SamacSys_Parts:1849535")
     )
     (path "/9cbbd2f9-4f34-4463-9a32-909d576e26a4"
-      (reference "J2") (unit 1) (value "Conn_01x04") (footprint "Connector_PinHeader_1.00mm:PinHeader_1x04_P1.00mm_Vertical")
+      (reference "J2") (unit 1) (value "Conn_01x04") (footprint "Connector_PinHeader_2.00mm:PinHeader_1x04_P2.00mm_Vertical")
     )
     (path "/1fcb31a2-51e4-4be3-8124-9d26e186cfb4/d6f246fc-9543-4b53-9a27-bdd4011ecf10"
@@
     )
     (path "/1fcb31a2-51e4-4be3-8124-9d26e186cfb4/fdabd193-05b7-418b-b423-c7f9635f8ada"
-      (reference "J10") (unit 1) (value "1-84953-5") (footprint "project_footprints:1849535")
+      (reference "J10") (unit 1) (value "1-84953-5") (footprint "SamacSys_Parts:1849535")
     )
     (path "/c779e344-5031-4f2d-bf31-77741b3c4be9/6bc05e1a-95ef-48ed-abfb-e1f927b61969"
@@
     )
     (path "/24bd5701-0eb0-4ec6-b68f-934ea2fa56bc/458d42de-4555-4a2d-af89-71f8f7dc5438"
-      (reference "R20") (unit 1) (value "10k") (footprint "Resistor_SMD:R_0603_1608Metric_Pad0.98x0.95mm_HandSolder")
+      (reference "R20") (unit 1) (value "10k") (footprint "Resistor_SMD:R_0805_2012Metric_Pad1.20x1.40mm_HandSolder")
     )
     (path "/c779e344-5031-4f2d-bf31-77741b3c4be9/4cf52119-fb49-4b3c-a2aa-682a95187367"
@@
     )
     (path "/c96310d5-5754-4cd6-8de7-7840ff32f085/458d42de-4555-4a2d-af89-71f8f7dc5438"
-      (reference "R22") (unit 1) (value "10k") (footprint "Resistor_SMD:R_0603_1608Metric_Pad0.98x0.95mm_HandSolder")
+      (reference "R22") (unit 1) (value "10k") (footprint "Resistor_SMD:R_0805_2012Metric_Pad1.20x1.40mm_HandSolder")
     )
     (path "/c779e344-5031-4f2d-bf31-77741b3c4be9/e887517c-961e-44c6-992b-959f9f108523"
@@
     )
     (path "/24bd5701-0eb0-4ec6-b68f-934ea2fa56bc/b1042786-9ebd-475f-a27d-633d437acdad"
-      (reference "R28") (unit 1) (value "1M") (footprint "Resistor_SMD:R_0603_1608Metric_Pad0.98x0.95mm_HandSolder")
+      (reference "R28") (unit 1) (value "1M") (footprint "Resistor_SMD:R_0805_2012Metric_Pad1.20x1.40mm_HandSolder")
     )
     (path "/c96310d5-5754-4cd6-8de7-7840ff32f085/b1042786-9ebd-475f-a27d-633d437acdad"
-      (reference "R29") (unit 1) (value "1M") (footprint "Resistor_SMD:R_0603_1608Metric_Pad0.98x0.95mm_HandSolder")
+      (reference "R29") (unit 1) (value "1M") (footprint "Resistor_SMD:R_0805_2012Metric_Pad1.20x1.40mm_HandSolder")
     )
     (path "/d7dab0b1-a885-42c4-b558-97d79e73318c/1214ef73-e2b5-465e-9b9d-b232033a9171"

Commit message: Some bugfixing, added cam.py script
Parts:
- J6: MouserNr (none) -> 538-50-36-1798
