File: CarPiPowerHat/CarPiPowerHat.kicad_pcb (KiCad board)
At the start: 4 copper layers, 96 x 85 mm, 115 parts, among them IC2 BD2226G-TR, J1 1-84953-5, J10 1-84953-5, J11 Conn_01x06_Male, J2 Conn_01x04, J3 HDMI_A_1.4, J4 AudioJack2_Ground, J5 HDMI_A_1.4, J6 Conn_02x03_Counter_Clockwise, J7 USB_A, J8 Conn_01x02_Male, J9 40HAT, Q3 DMG2305, Q4 DMP3013SFV-7, U1 PCF85063AT/AAZ, U2 ATtiny45V-20SU, U3 AP64501SP-13, U4 CAT24C32, U5 XC6206P332MR, U6 UDA1334ATS, U7 LM3480-5.0, Y1 FC-12M32.768KHZ7PF20PPM

Commit message: Finalizing, checking parts
Might be ready for production
Parts:
- C38: footprint Capacitor_SMD:C_0603_1608Metric_Pad1.08x0.95mm_HandSolder -> Capacitor_SMD:C_1206_3216Metric_Pad1.33x1.80mm_HandSolder
- J1, J10: footprint project_footprints:1849535 -> SamacSys_Parts:1849535
- J2: footprint Connector_PinHeader_1.00mm:PinHeader_1x04_P1.00mm_Vertical -> Connector_PinHeader_2.00mm:PinHeader_1x04_P2.00mm_Vertical
- R20, R22, R28, R29: footprint Resistor_SMD:R_0603_1608Metric_Pad0.98x0.95mm_HandSolder -> Resistor_SMD:R_0805_2012Metric_Pad1.20x1.40mm_HandSolder
- moved IC2 3.93 mm to (142.5, 95.3), turned to -90 degrees
- moved C38 3.75 mm to (140.2, 92.0), turned to 180 degrees
- moved R28 3.07 mm to (151.9, 79.0), turned to 0 degrees
- moved R29 3.04 mm to (151.9, 83.3), turned to 0 degrees
- moved F2 2.63 mm to (167.2, 91.2)
- moved J2 2.17 mm to (80.8, 97.3)
- moved C39 1.72 mm to (144.4, 92.0)
- moved D8 1.63 mm to (165.2, 84.6)
- moved C29 0.90 mm to (153.3, 89.0)
- moved D4 0.90 mm to (153.3, 86.7)
- moved R20 0.90 mm to (152.3, 92.2)
- moved C21 0.70 mm to (112.5, 72.6)
- moved C24 0.70 mm to (114.3, 72.8)
- moved C9 0.16 mm to (167.0, 38.5)
Connections:
- net /PSU/+5v renamed /Raspberry Pi/P5V_HAT
Routing:
- net GND: track 125.0 -> 133.0 mm, vias 258 -> 280
- net /PSU/USB_5v: track 30.9 -> 26.5 mm
- net /Raspberry Pi/BCM25: track 45.3 -> 42.3 mm
- net /+12v: track 6.06 -> 8.71 mm
- net Net-(C33-Pad1): track 26.7 -> 24.1 mm
- net Net-(C21-Pad1): track 22.0 -> 24.0 mm
- net /HDMI Connector Camera/D: track 9.69 -> 11.6 mm
- net /Raspberry Pi/P5V_HAT: track 181.6 -> 180.0 mm
- net /+3.3v: track 118.4 -> 119.4 mm
- net /HDMI Connector Camera/C: track 8.63 -> 9.62 mm
- net /Light Input/OUT: track 45.2 -> 44.3 mm
- net /i2s_dac/VREF: track 7.73 -> 8.56 mm
- net PWR_SENSE_OUT: track 124.1 -> 124.9 mm
- added copper zone on F.Cu, net /PSU/USB_5v
Other:
- board text added: "A"
- board text added: "B"
- board text added: "C"
- board text added: "D"
- board text added: "Power 1A"
- board text removed: "D C B A"
- board text removed: "Power"
