File: CarPiPowerHat/hdmi_connectors.kicad_sch (KiCad schematic)
At the start: 2 parts, among them J10 1-84953-5, J3 HDMI_A_1.4

Commit message: Moved HDMI ports
The HDMI ports were offset by 1-2 mm
Parts:
- renumbered J10 to J1, J3 to J5
Changed lines of the file:
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@@
   (symbol (lib_id "1-84953-5:1-84953-5") (at 45.72 30.48 0)
     (in_bom yes) (on_board yes)
-    (property "Reference" "J10" (id 0) (at 58.42 24.13 0))
+    (property "Reference" "J1" (id 0) (at 58.42 24.13 0))
     (property "Value" "1-84953-5" (id 1) (at 58.42 26.67 0))
     (property "Footprint" "SamacSys_Parts:1849535" (id 2) (at 67.31 27.94 0)
@@
   (symbol (lib_id "CarPiPowerHat:HDMI_A_1.4") (at 186.69 49.53 0)
     (in_bom yes) (on_board yes)
-    (property "Reference" "J3" (id 0) (at 191.77 22.86 0)
+    (property "Reference" "J5" (id 0) (at 191.77 22.86 0)
       (effects (font (size 1.27 1.27)) (justify left))
     )
