File: CarPiPowerHat/raspberry.kicad_sch (KiCad schematic)
At the start: 6 parts, among them J3 40HAT, U2 CAT24C32

Commit message: Finalizing
Parts:
- removed R2: DNP, project_footprints:R_0603_1608Metric_Pad0.84x1.00mm_HandSolder, symbol Device:R
- added JP1: SolderJumper_2_Open, Jumper:SolderJumper-2_P1.3mm_Open_RoundedPad1.0x1.5mm, symbol Jumper:SolderJumper_2_Open
Connections:
- net GND: now also JP1.1 (A)
- net at R3.2, U2.7 (WP): now also JP1.2 (B)
Changed lines of the file:
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@@
     (pin "1")
   )
-  (symbol (lib_id "Device:R") (at 62.865 147.32 270) (unit 1)
+  (symbol (lib_id "Jumper:SolderJumper_2_Open") (at 62.865 147.32 0) (unit 1)
     (in_bom yes) (on_board yes)
-    (property "Reference" "R2" (id 0) (at 62.865 149.352 90))
-    (property "Value" "DNP" (id 1) (at 62.865 147.32 90))
-    (property "Footprint" "project_footprints:R_0603_1608Metric_Pad0.84x1.00mm_HandSolder" (id 2) (at 62.865 145.542 90)
+    (property "Reference" "JP1" (id 0) (at 62.865 144.78 0))
+    (property "Value" "SolderJumper_2_Open" (id 1) (at 46.355 147.955 0)
       (effects (font (size 1.27 1.27)) hide)
     )
+    (property "Footprint" "Jumper:SolderJumper-2_P1.3mm_Open_RoundedPad1.0x1.5mm" (id 2) (at 62.865 147.32 0)
+      (effects (font (size 1.27 1.27)) hide)
+    )

Commit message: Added part numbers
* Selected parts from lcsc
* Checked footprints
Parts:
- R3: LCSC C25804 -> C25804
- R6, R8: LCSC C22978 -> C23018
- U2: LCSC (none) -> C81193
Other:
- title: (none) -> Raspberry Pi Header
Changed lines of the file:
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@@
 (kicad_sch (version 20210621) (generator eeschema)
   (paper "A4")
+  (title_block
+    (title "Raspberry Pi Header")
+    (date "2021-08-24")
+    (rev "1")
+  )
   (junction (at 63.5 137.16) (diameter 1.016) (color 0 0 0 0))
   (junction (at 63.5 139.7) (diameter 1.016) (color 0 0 0 0))
@@
       (effects (font (size 1.27 1.27)) hide)
     )
-    (property "LCSC" " C25804" (id 4) (at 69.85 152.4 90)
+    (property "LCSC" "C25804" (id 4) (at 69.85 152.4 90)
       (effects (font (size 1.27 1.27)) hide)
     )
@@
       (effects (font (size 1.27 1.27)) hide)
     )
-    (property "LCSC" "C22978" (id 4) (at 90.17 181.61 90)
+    (property "LCSC" "C23018" (id 4) (at 90.17 181.61 90)
       (effects (font (size 1.27 1.27)) hide)
     )
@@
       (effects (font (size 1.27 1.27)) hide)
     )
-    (property "LCSC" "C22978" (id 4) (at 90.17 187.96 90)
+    (property "LCSC" "C23018" (id 4) (at 90.17 187.96 90)
       (effects (font (size 1.27 1.27)) hide)
     )
@@
     (property "Footprint" "Package_SOIC:SOIC-8_3.9x4.9mm_P1.27mm" (id 2) (at 107.95 153.035 0))
     (property "Datasheet" "" (id 3) (at 83.82 142.24 0))
+    (property "LCSC" "C81193" (id 4) (at 83.82 142.24 0)
+      (effects (font (size 1.27 1.27)) hide)
+    )
     (pin "4")
     (pin "8")

Commit message: Fixed some bugs, not done yet
Parts:
- renumbered J3 to J9, R8 to R13, R6 to R14, R3 to R17, U2 to U4
Changed lines of the file:
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@@
   (symbol (lib_id "Device:R") (at 69.85 152.4 180) (unit 1)
     (in_bom yes) (on_board yes)
-    (property "Reference" "R3" (id 0) (at 67.818 152.4 90))
+    (property "Reference" "R17" (id 0) (at 67.818 152.4 90))
     (property "Value" "10K" (id 1) (at 69.85 152.4 90))
     (property "Footprint" "Resistor_SMD:R_0603_1608Metric" (id 2) (at 71.628 152.4 90)
@@
   (symbol (lib_id "Device:R") (at 90.17 181.61 270) (unit 1)
     (in_bom yes) (on_board yes)
-    (property "Reference" "R6" (id 0) (at 90.17 183.642 90))
+    (property "Reference" "R14" (id 0) (at 90.17 183.642 90))
     (property "Value" "3.9K" (id 1) (at 90.17 181.61 90))
     (property "Footprint" "Resistor_SMD:R_0603_1608Metric" (id 2) (at 90.17 179.832 90)
@@
   (symbol (lib_id "Device:R") (at 90.17 187.96 270) (unit 1)
     (in_bom yes) (on_board yes)
-    (property "Reference" "R8" (id 0) (at 90.17 189.992 90))
+    (property "Reference" "R13" (id 0) (at 90.17 189.992 90))
     (property "Value" "3.9K" (id 1) (at 90.17 187.96 90))
     (property "Footprint" "Resistor_SMD:R_0603_1608Metric" (id 2) (at 90.17 186.182 90)
@@
   (symbol (lib_id "CarPiPowerHat:CAT24C32") (at 83.82 142.24 0) (unit 1)
     (in_bom yes) (on_board yes)
-    (property "Reference" "U2" (id 0) (at 92.71 133.35 0))
+    (property "Reference" "U4" (id 0) (at 92.71 133.35 0))
     (property "Value" "CAT24C32" (id 1) (at 77.47 133.35 0))
     (property "Footprint" "Package_SOIC:SOIC-8_3.9x4.9mm_P1.27mm" (id 2) (at 107.95 153.035 0))
@@
   (symbol (lib_id "CarPiPowerHat:OX40HAT") (at 91.44 46.355 0) (unit 1)
     (in_bom yes) (on_board yes)
-    (property "Reference" "J3" (id 0) (at 100.33 43.815 0))
+    (property "Reference" "J9" (id 0) (at 100.33 43.815 0))
     (property "Value" "40HAT" (id 1) (at 83.82 43.815 0))
     (property "Footprint" "Connector_PinSocket_2.54mm:PinSocket_2x20_P2.54mm_Vertical" (id 2) (at 91.44 41.275 0)
