File: CarPiPowerHat/CarPiPowerHat-backups/input_pin_protect.kicad_sch (KiCad schematic)
At the start: 7 parts

Commit message: Repositioning of connectors
Parts:
- D11: footprint Diode_SMD:D_0603_1608Metric -> (none)
Changed lines of the file:
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@@
       (effects (font (size 1.27 1.27)) (justify right))
     )
-    (property "Footprint" "Diode_SMD:D_0603_1608Metric" (id 2) (at 138.43 86.36 0)
+    (property "Footprint" "" (id 2) (at 138.43 86.36 0)
       (effects (font (size 1.27 1.27)) hide)
     )
