File: CarPiPowerHat/CarPiPowerHat-backups/power_control.kicad_sch (KiCad schematic)
At the start: 21 parts, among them U3 LM3480-5.0, U4 ATtiny45V-10X

Commit message: Repositioning of connectors
Connections:
- net IGN: now also C20.1, D5.2 (A2), F2.2, U3.2 (VI)
- net +5v renamed P5V_HAT
Changed lines of the file:
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@@
+    (effects (font (size 1.27 1.27)) (justify right bottom))
+  )
+  (label "IGN" (at 51.435 43.815 180)
     (effects (font (size 1.27 1.27)) (justify right bottom))
   )
@@
     )
   )
-  (hierarchical_label "+5v" (shape input) (at 26.67 31.115 180)
+  (hierarchical_label "P5V_HAT" (shape input) (at 26.67 31.115 180)
     (effects (font (size 1.27 1.27)) (justify right))
   )
